File: memory_pcb/memory_pcb.kicad_pcb (KiCad board)
At the start: 2 copper layers, 110 x 54 mm, 70 parts, among them J1 Conn_01x10, P1 AFC01-S10FCC-00, SW1 SW_Push, SW2 SW_Push, U1 AP3602AKTR-G1 SETUPUP, U10 DMG3415U, U11 SS54_C22452, U12 TYPE-C-31-M-12, U2 ESP32-S3-WROOM-1(N16R8), U3 100SP3T2B4M6RE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

Commit message: uz nevim, dneska asi konec
Parts:
- removed C5: 1uF, new_lib_footprint:C1206
- added C17: 1uF 0603, new_lib_footprint:C0603, F.Cu at (115.6, 59.0)
- moved C10 87.5 mm to (109.2, 64.7), turned to 180 degrees
- moved C3 86.1 mm to (110.1, 71.2), turned to 90 degrees
- moved U1 86.0 mm to (109.2, 68.0), turned to -90 degrees
- moved U10 84.9 mm to (105.2, 65.5), turned to -90 degrees
- moved C9 84.4 mm to (117.8, 59.2), turned to 90 degrees
- moved C4 83.5 mm to (108.2, 71.2), turned to 90 degrees
- moved C1 82.1 mm to (106.7, 71.2), turned to -90 degrees
- moved C7 76.8 mm to (99.4, 61.6), turned to -90 degrees
- moved R6 76.7 mm to (99.3, 64.7), turned to 90 degrees
- moved C8 76.4 mm to (105.3, 62.0)
- moved U9 76.4 mm to (102.2, 63.0)
- moved U11 75.5 mm to (101.8, 68.4), turned to -90 degrees
- moved C12 75.3 mm to (104.7, 71.2), turned to 90 degrees
- moved U6 74.0 mm to (109.2, 62.6), turned to -90 degrees
- moved C13 73.4 mm to (102.4, 72.8)
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Routing:
- net VBUS: track 12.5 -> 77.7 mm, vias 0 -> 2
- net /RESET: track 4.02 -> 66.5 mm, vias 0 -> 3
- net /BOOT: track 0.00 -> 57.8 mm, vias 0 -> 2
- net GND: track 11.0 -> 67.6 mm, vias 0 -> 15
- net Net-(LED1-K): track 0.00 -> 51.1 mm, vias 0 -> 2
- net VBAT: track 1.35 -> 49.7 mm, vias 0 -> 2
- net +3.3V: track 35.7 -> 75.6 mm, vias 0 -> 2
- net +5V: track 6.48 -> 46.3 mm, vias 0 -> 2
- net /CLK: track 5.16 -> 39.6 mm, vias 0 -> 2
- net Net-(R17-Pad2): track 0.00 -> 33.0 mm, vias 0 -> 2
- net Net-(R16-Pad2): track 9.22 -> 32.3 mm
- net /DISP_CS: track 10.4 -> 31.9 mm, vias 1 -> 2
- net /ENC_BTN: track 3.03 -> 18.8 mm, vias 0 -> 2
- net /SCL: track 1.95 -> 15.2 mm, vias 0 -> 2
- net /SDA: track 1.93 -> 14.8 mm, vias 0 -> 2
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Other:
- board text added: "ESP32 economic vias around for GND general capatiors where"

Commit message: proc je tu tolik filu
Parts:
- U5: value BOOT -> TS-1088-AR02016
Routing:
- net /BOOT: track 57.8 -> 59.5 mm
- net Net-(ENC1-PadS1): track 54.8 -> 53.3 mm
- net +3.3V: track 75.6 -> 77.1 mm, vias 2 -> 0
- net VBAT: track 49.7 -> 50.4 mm, vias 2 -> 4
- net GND: vias 15 -> 17
Other:
- board text added: "ESP32 economic vias around for GND general capatiors where esp anthena economic assembly"
- board text removed: "ESP32 economic vias around for GND general capatiors where"

Commit message: im sleeping
Parts:
- moved J1 74.0 mm to (149.4, 101.0), turned to -90 degrees
- moved SW2 1.62 mm to (149.0, 87.0)
- moved SW1 0.78 mm to (149.0, 68.0)
Connections:
- J1 pad 10: /48 -> /21
- J1 pad 8: /21 -> /48
Routing:
- net +5V: track 46.5 -> 23.4 mm
- net +3.3V: track 77.1 -> 64.4 mm
- net /21: track 39.9 -> 27.4 mm, vias 2 -> 0
- net /47: track 38.8 -> 26.8 mm, vias 2 -> 0
- net /02: track 33.1 -> 45.1 mm
- net /48: track 37.7 -> 28.0 mm, vias 2 -> 0
- net /01: track 37.1 -> 44.8 mm, vias 2 -> 0
- net /RX: track 40.2 -> 44.3 mm, vias 0 -> 2
- net Net-(R16-Pad2): track 32.3 -> 34.6 mm
- net /TX: track 43.0 -> 44.2 mm
- net Net-(R17-Pad2): track 33.0 -> 33.9 mm

Commit message: looks rdy
Parts:
- removed C12: 1uF, new_lib_footprint:C1206
- added C5: 1uF 0603, new_lib_footprint:C0603, F.Cu at (80.3, 70.3)
- added TP1: D+, TestPoint:TestPoint_Pad_D1.0mm, F.Cu at (69.4, 101.1)
- added TP2: D-, TestPoint:TestPoint_Pad_D1.0mm, F.Cu at (69.4, 96.3)
- R10, R11, R12, R13, R14, R15, R3, R8, R9: value 5.1kOhm -> 10kOhm
- moved J1 54.3 mm to (95.1, 101.0)
- moved R4 26.1 mm to (72.4, 70.0), turned to 180 degrees
- moved C16 25.2 mm to (84.5, 74.1), turned to 0 degrees
- moved R5 25.0 mm to (72.5, 61.4), turned to 0 degrees
- moved C1 24.1 mm to (82.6, 71.2)
- moved C10 24.1 mm to (85.1, 64.7)
- moved C11 24.1 mm to (88.1, 62.9)
- moved C14 24.1 mm to (94.3, 70.3)
- moved C15 24.1 mm to (94.3, 73.5)
- moved C17 24.1 mm to (91.5, 59.0)
- moved C2 24.1 mm to (94.3, 66.8)
- moved C3 24.1 mm to (86.0, 71.2)
- moved C7 24.1 mm to (75.3, 61.6)
- moved C8 24.1 mm to (81.2, 62.0)
- moved R10 24.1 mm to (88.8, 66.9)
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- renumbered U5 to SW1, U4 to SW2, SW1 to SW3, SW2 to SW4, U3 to SW5
Connections:
- net /RESET renamed Net-(U2-EN)
- SW1 pad 1: GND -> Net-(U2-IO0)
- SW1 pad 2: /BOOT -> GND
- U2 pad 27: /BOOT -> Net-(U2-IO0)
Routing:
- net /BOOT: track 59.5 -> 0.00 mm, vias 2 -> 0
- net /21: track 27.4 -> 71.5 mm
- net /47: track 26.8 -> 68.9 mm
- net +5V: track 23.4 -> 64.9 mm
- net /48: track 28.0 -> 66.0 mm
- net +3.3V: track 64.4 -> 100.7 mm, vias 0 -> 3
- net Net-(U2-IO0): track 0.00 -> 32.9 mm, vias 0 -> 2
- net /02: track 45.1 -> 77.3 mm
- net /01: track 44.8 -> 76.2 mm
- net /RX: track 44.3 -> 75.0 mm
- net /TX: track 44.2 -> 74.4 mm
- net GND: track 67.6 -> 41.9 mm, vias 17 -> 28
- net /D+: track 80.7 -> 55.3 mm, vias 2 -> 0
- net Net-(ENC1-PadA): track 68.1 -> 44.0 mm
- net Net-(ENC1-PadS1): track 53.3 -> 29.1 mm
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Other:
- board text added: "ESP32 economic vias around for GND ground under D+ D- x general capatiors where x esp anthena economic assembly"
- board text removed: "ESP32 economic vias around for GND general capatiors where esp anthena economic assembly"

Commit message: :)
Parts:
- added C12: 0.1uF, new_lib_footprint:C0402, F.Cu at (123.7, 84.9)
- added C18: 0.1uF, new_lib_footprint:C0402, F.Cu at (107.4, 80.8)
- added C19: 1uF 0603, new_lib_footprint:C0603, F.Cu at (127.2, 85.2)
- moved LED1 7.25 mm to (59.1, 93.7)
Connections:
- JP5 pad 1: +5V -> /DISP_ON
- JP7 pad 1: +5V -> unconnected-(JP7-A-Pad1)
- JP8 pad 1: GND -> unconnected-(JP8-A-Pad1)
- U2 pad 31: unconnected-(U2-IO38-Pad31) -> /DISP_ON
Routing:
- net /DISP_ON: track 0.00 -> 17.8 mm, vias 0 -> 2
- net Net-(LED1-K): track 34.3 -> 41.5 mm, vias 2 -> 0
- net +5V: track 64.9 -> 62.0 mm
- net GND: vias 28 -> 31

Commit message: a
Parts:
- moved C12 22.9 mm to (101.3, 80.4)
- moved C19 21.6 mm to (106.2, 79.9), turned to 180 degrees
- moved JP12 19.1 mm to (71.5, 57.7), turned to 0 degrees
- moved JP11 10.3 mm to (71.5, 60.2), turned to 0 degrees
- moved R5 9.90 mm to (72.2, 71.3), turned to 180 degrees
- moved R4 6.41 mm to (70.9, 63.7), turned to 90 degrees
- moved C6 5.54 mm to (72.5, 69.9), turned to 0 degrees
- moved C18 1.80 mm to (109.2, 80.5), turned to 180 degrees
- moved JP1 0.80 mm to (93.8, 82.8)
- moved JP10 0.80 mm to (116.2, 82.8)
- moved JP2 0.80 mm to (96.2, 82.8)
- moved JP3 0.80 mm to (98.8, 82.8)
- moved JP4 0.80 mm to (101.2, 82.8)
- moved JP5 0.80 mm to (103.8, 82.8)
- moved JP6 0.80 mm to (106.2, 82.8)
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Connections:
- JP7 pad 1: unconnected-(JP7-A-Pad1) -> +5V
- JP8 pad 1: unconnected-(JP8-A-Pad1) -> GND
Routing:
- net Net-(JP12-A): track 3.66 -> 16.4 mm
- net GND: track 41.9 -> 31.0 mm, vias 31 -> 20
- net Net-(LED1-K): track 41.5 -> 32.7 mm, vias 0 -> 2
- net Net-(JP11-A): track 3.66 -> 8.62 mm
- net Net-(ENC1-PadA): track 44.0 -> 39.5 mm
- net /PWR_SW: track 50.9 -> 47.6 mm
- net VBAT: track 37.0 -> 33.7 mm
- net Net-(ENC1-PadB): track 41.3 -> 39.4 mm
- net /DISP_ON: track 17.8 -> 19.3 mm
- net Net-(U7-STAT): track 4.61 -> 3.09 mm
- net Net-(ENC1-PadS1): track 29.1 -> 30.4 mm
- net VBUS: track 55.7 -> 54.7 mm
- net /DISP_CS: track 8.03 -> 7.23 mm
- net Net-(JP7-B): track 6.20 -> 7.00 mm
- net Net-(JP6-B): track 5.37 -> 6.17 mm
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Other:
- outline, holes or cut-outs redrawn

Commit message: posilam
Parts:
- removed TP1: D+, TestPoint:TestPoint_Pad_D1.0mm
- removed TP2: D-, TestPoint:TestPoint_Pad_D1.0mm
- moved R17 30.8 mm to (120.2, 65.7), turned to -90 degrees
- moved C11 29.2 mm to (117.2, 65.2)
- moved R12 27.6 mm to (118.6, 65.7), turned to -90 degrees
- moved R16 27.4 mm to (120.2, 69.2), turned to 90 degrees
- moved R11 27.4 mm to (118.6, 69.2), turned to 90 degrees
- moved C2 23.1 mm to (117.2, 69.8)
- moved JP12 18.3 mm to (53.8, 62.3), turned to 180 degrees
- moved JP11 17.7 mm to (53.8, 59.8), turned to 180 degrees
- moved R4 16.7 mm to (82.0, 76.2), turned to 180 degrees
- moved R5 13.5 mm to (85.0, 75.3), turned to 90 degrees
- moved C13 13.1 mm to (83.3, 59.8)
- moved C6 12.8 mm to (85.0, 72.7), turned to 90 degrees
- moved U7 12.1 mm to (82.3, 73.2), turned to 90 degrees
- moved R6 9.80 mm to (84.7, 67.2), turned to 0 degrees
- moved C5 9.38 mm to (83.0, 61.3), turned to 180 degrees
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Connections:
- J1 pad 2: +3.3V -> +5V
- J1 pad 3: +5V -> +3.3V
Routing:
- net Net-(U2-EN): track 45.1 -> 92.7 mm, vias 3 -> 4
- net Net-(R17-Pad2): track 56.0 -> 25.2 mm
- net Net-(R16-Pad2): track 56.7 -> 29.1 mm
- net /BTN2: track 5.40 -> 27.1 mm, vias 0 -> 2
- net Net-(U2-IO0): track 32.9 -> 47.9 mm
- net GND: track 31.0 -> 20.0 mm, vias 20 -> 19
- net /BTN1: track 15.7 -> 25.9 mm
- net Net-(JP12-A): track 16.4 -> 6.51 mm
- net Net-(JP11-A): track 8.62 -> 15.8 mm
- net /02: track 77.3 -> 84.3 mm
- net /01: track 76.2 -> 83.2 mm
- net +3.3V: track 100.7 -> 107.6 mm, vias 3 -> 5
- net VBAT: track 33.7 -> 39.6 mm, vias 5 -> 4
- net Net-(LED1-K): track 32.7 -> 38.6 mm
- net /48: track 65.8 -> 71.2 mm
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
Commit message: step1
Parts:
- moved C17 1.19 mm to (92.6, 58.7), turned to -90 degrees
- moved C9 0.40 mm to (91.0, 59.2), turned to 90 degrees
Routing:
- net GND: track 20.0 -> 18.3 mm
- net Net-(U2-EN): track 92.7 -> 92.2 mm
