File: memory_pcb/memory_pcb_backup1.kicad_pcb (KiCad board)
At the start: 2 copper layers, 110 x 54 mm, 70 parts, among them J1 Conn_01x10, P1 AFC01-S10FCC-00, SW1 SW_Push, SW2 SW_Push, U1 AP3602AKTR-G1 SETUPUP, U10 DMG3415U, U11 SS54_C22452, U12 TYPE-C-31-M-12, U2 ESP32-S3-WROOM-1(N16R8), U3 100SP3T2B4M6RE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

Commit message: prvni cena test
Parts:
- JP4: value EXTC -> EXTCOM
- JP8: value EXTM -> EXTMOD
Routing:
- net /MOSI: track 32.8 -> 5.87 mm, vias 2 -> 0
- net /PWR_SW: track 69.2 -> 55.9 mm
- net /DISP_CS: track 10.4 -> 5.28 mm, vias 1 -> 0
- net /CLK: track 5.16 -> 7.60 mm
- net /48: track 37.7 -> 36.7 mm
- net /47: track 38.8 -> 38.2 mm
