File: memory_pcb/memory_pcb_backup2.kicad_pcb (KiCad board)
At the start: 2 copper layers, 110 x 54 mm, 70 parts, among them J1 Conn_01x10, P1 AFC01-S10FCC-00, SW1 SW_Push, SW2 SW_Push, U1 AP3602AKTR-G1 SETUPUP, U10 DMG3415U, U11 SS54_C22452, U12 TYPE-C-31-M-12, U2 ESP32-S3-WROOM-1(N16R8), U3 100SP3T2B4M6RE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

Commit message: prvni cena test
Parts:
- removed C5: 1uF, new_lib_footprint:C1206
- added C17: 1uF 0603, new_lib_footprint:C0603, F.Cu at (115.6, 59.0)
- moved U10 61.2 mm to (86.6, 84.1), turned to -90 degrees
- moved U8 54.4 mm to (76.9, 56.4)
- moved R3 53.4 mm to (115.6, 60.7), turned to 0 degrees
- moved R6 52.8 mm to (80.7, 83.3), turned to 90 degrees
- moved C7 52.7 mm to (80.8, 80.2), turned to -90 degrees
- moved U9 52.3 mm to (83.6, 81.6)
- moved C8 52.3 mm to (86.7, 80.6)
- moved U11 51.7 mm to (83.2, 87.0), turned to -90 degrees
- moved R7 43.9 mm to (80.0, 87.0), turned to 0 degrees
- moved U5 24.3 mm to (95.7, 100.9), turned to -90 degrees
- moved U4 12.3 mm to (89.3, 100.9), turned to -90 degrees
- moved R2 0.36 mm to (64.2, 93.5)
- moved R1 0.32 mm to (61.5, 93.5)
- turned C14 to -90 degrees
Connections:
- J1 pad 4: /TX -> /RX
- J1 pad 5: /RX -> /TX
Routing:
- net /CLK: track 5.16 -> 39.6 mm, vias 0 -> 2
- net Net-(R17-Pad2): track 0.00 -> 33.0 mm, vias 0 -> 2
- net VBUS: track 12.5 -> 41.6 mm
- net Net-(R16-Pad2): track 9.22 -> 32.3 mm
- net /DISP_CS: track 10.4 -> 31.9 mm, vias 1 -> 2
- net /ENC_BTN: track 3.03 -> 18.8 mm, vias 0 -> 2
- net /D-: track 90.6 -> 80.6 mm, vias 2 -> 0
- net GND: track 11.0 -> 20.4 mm, vias 0 -> 2
- net /RESET: track 4.02 -> 12.5 mm, vias 0 -> 2
- net /D+: track 87.7 -> 80.7 mm, vias 0 -> 2
- net +3.3V: track 35.7 -> 38.4 mm
- net /ALRT: track 12.7 -> 14.7 mm
- net /PWR_SW: track 69.2 -> 70.7 mm
- net /MOSI: track 32.8 -> 34.1 mm
- net Net-(ENC1-PadB): track 64.5 -> 65.4 mm
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