File: memory_pcb/inputs.kicad_sch (KiCad schematic)
At the start: 12 parts, among them SW1 SW_Push, SW2 SW_Push, SW3 RotaryEncoder_Switch, U3 100SP3T2B4M6RE

Commit message: and so it begins
Parts:
- added C11, C14, C15, C16, C2: 0.1uF, new_lib_footprint:C0402, symbol new_lib_symbol:CL05B104KO5NNNC
- added R16, R17, R18, R19, R20: 1kOhm, new_lib_footprint:R0603, symbol new_lib_symbol:0603WAF1001T5E
- ENC1: renamed from SW3; footprint (none) -> Rotary_Encoder:RotaryEncoder_Alps_EC11E-Switch_Vertical_H20mm; now not fitted
- U3: footprint new_lib_footprint:SW-TH_100SP3T2B4M6RE -> new_lib_footprint:MTS-102-C3
Connections:
- net BTN1: now also C11.2, R17.1; no longer SW1.1
- net BTN2: now also C2.2, R16.1; no longer SW2.1
- net ENC_BTN: now also C16.2, R20.2; no longer ENC1.S1
- net ENC_SIG_A: now also C14.2, R18.1; no longer ENC1.A
- net ENC_SIG_B: now also C15.2, R19.1; no longer ENC1.B
- net GND: now also C11.1, C14.1, C15.1, C16.1, C2.1
- new net: ENC1.B, R19.2
- new net: ENC1.S1, R20.1
- new net: R17.2, SW1.1
- new net: ENC1.A, R18.2
- new net: R16.2, SW2.1
Other:
- moved on the sheet: R11, R12, R13, R14, R15, SW1, SW2

Commit message: looks rdy
Parts:
- R10, R11, R12, R13, R14, R15: value 5.1kOhm -> 10kOhm; LCSC C23186 -> C25804
- renumbered SW1 to SW3, SW2 to SW4, U3 to SW5
Changed lines of the file:
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@@
 			)
 		)
-		(property "Value" "5.1kOhm"
+		(property "Value" "10kOhm"
 			(at 78.74 30.4801 90)
 			(effects
@@
 			)
 		)
-		(property "LCSC" "C23186"
+		(property "LCSC" "C25804"
 			(at 81.28 31.75 0)
 			(effects
@@
 			)
 		)
-		(property "Value" "5.1kOhm"
+		(property "Value" "10kOhm"
 			(at 218.44 76.1999 90)
 			(effects
@@
 			)
 		)
-		(property "LCSC" "C23186"
+		(property "LCSC" "C25804"
 			(at 215.9 74.93 0)
 			(effects
@@
 			)
 		)
-		(property "Value" "5.1kOhm"
+		(property "Value" "10kOhm"
 			(at 161.798 76.2 90)
 			(effects
@@
 			)
 		)
-		(property "LCSC" "C23186"
+		(property "LCSC" "C25804"
 			(at 160.02 74.93 0)
 			(effects
@@
 			)
 		)
-		(property "Value" "5.1kOhm"
+		(property "Value" "10kOhm"
 			(at 143.764 76.2 90)
 			(effects
@@
 			)
 		)
-		(property "LCSC" "C23186"
+		(property "LCSC" "C25804"
 			(at 153.67 74.93 0)
 			(effects
@@
 		(dnp yes)
 		(fields_autoplaced yes)
-		(property "Reference" "U3"
+		(property "Reference" "SW5"
 			(at 86.36 104.14 0)
 			(effects
@@
 			(project "memory_pcb"
 				(path "/0b554bab-2912-44e0-8d16-f1690413cb05/0b536339-25e4-48ce-a11a-b22c2b02a50f"
-					(reference "U3")
+					(reference "SW5")
 					(unit 1)
 				)
@@
 			)
 		)
-		(property "Value" "5.1kOhm"
+		(property "Value" "10kOhm"
 			(at 72.39 104.1399 90)
 			(effects
@@
 			)
 		)
-		(property "LCSC" "C23186"
+		(property "LCSC" "C25804"
 			(at 69.85 102.87 0)
 			(effects
@@
 		(dnp yes)
 		(fields_autoplaced yes)
-		(property "Reference" "SW1"
+		(property "Reference" "SW3"
 			(at 53.34 31.75 0)
 			(effects
@@
 			(project "memory_pcb"
 				(path "/0b554bab-2912-44e0-8d16-f1690413cb05/0b536339-25e4-48ce-a11a-b22c2b02a50f"
-					(reference "SW1")
+					(reference "SW3")
 					(unit 1)
 				)
@@
 		(dnp yes)
 		(fields_autoplaced yes)
-		(property "Reference" "SW2"
+		(property "Reference" "SW4"
 			(at 101.6 31.75 0)
 			(effects
@@
 			(project "memory_pcb"
 				(path "/0b554bab-2912-44e0-8d16-f1690413cb05/0b536339-25e4-48ce-a11a-b22c2b02a50f"
-					(reference "SW2")
+					(reference "SW4")
 					(unit 1)
 				)
@@
 			)
 		)
-		(property "Value" "5.1kOhm"
+		(property "Value" "10kOhm"
 			(at 30.48 30.4801 90)
 			(effects
@@
 			)
 		)
-		(property "LCSC" "C23186"
+		(property "LCSC" "C25804"
 			(at 33.02 31.75 0)
 			(effects
