File: memory_pcb/memory_pcb.kicad_sch (KiCad schematic)
At the start: 42 parts, among them P1 AFC01-S10FCC-00, U1 AP3602AKTR-G1 SETUPUP, U10 DMG3415U, U11 SS54_C22452, U2 ESP32-S3-WROOM-1(N16R8), U3 GT-USB-7047C, U4 TS-1088-AR02016, U5 TS-1088-AR02016, U6 MAX17048G+T10 FUEL GAUGE, U7 MCP73831T-2ACI/OT Charger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

Commit message: pondeli klasika
Parts:
- removed C2: 1uF, new_lib_footprint:C1206, symbol new_lib_symbol:CL31B105KBHNNNE
- removed U3: GT-USB-7047C, new_lib_footprint:USB-C-SMD_GT-USB-7047C, symbol new_lib_symbol:GT-USB-7047C
- added C10: 1uF 0603, new_lib_footprint:C0603, symbol new_lib_symbol:CL10A105KB8NNNC
- added C12: 1uF, new_lib_footprint:C1206, symbol new_lib_symbol:CL31B105KBHNNNE
- added C13: 0.1uF, new_lib_footprint:C0402, symbol new_lib_symbol:CL05B104KO5NNNC
- added C9: 10uF, new_lib_footprint:C0402, symbol new_lib_symbol:0402B102K500NT
- added R8, R9: 5.1kOhm, new_lib_footprint:R0603, symbol new_lib_symbol:0603WAF5101T5E
- added U12: TYPE-C-31-M-12, new_lib_footprint:USB-C_SMD-TYPE-C-31-M-12_1, symbol new_lib_symbol:TYPE-C-31-M-12
- H1, H2, H3, H4: footprint MountingHole:MountingHole_2.7mm_M2.5_Pad -> MountingHole:MountingHole_2.2mm_M2_DIN965_Pad
- JP1, JP10, JP2, JP3, JP4, JP5, JP6, JP7, JP8, JP9: footprint Jumper:SolderJumper-2_P1.3mm_Bridged_Pad1.0x1.5mm -> Jumper:SolderJumper-2_P1.3mm_Bridged_RoundedPad1.0x1.5mm
- U5: value TS-1088-AR02016 -> BOOT
Connections:
- net +3.3V: now also C12.2, C13.2, C9.1, R8.2, R9.2
- net D+: now also U12.A6 (DP1), U12.B6 (DP2)
- net D-: now also U12.A7 (DN1), U12.B7 (DN2)
- net GND: now also C12.1, C13.1, C9.2, U12.1 (EH), U12.2 (EH), U12.3 (EH), U12.4 (EH), U12.A1B12 (GND), U12.B1A12 (GND)
- net SCL: now also U2.5 (IO5), R9.1; no longer U2.4 (IO4)
- net SDA: now also U2.4 (IO4), R8.1; no longer U2.15 (IO3)
- net VBUS: now also U12.A4B9 (VBUS), U12.B4A9 (VBUS)
- net at R1.2: now also U12.A5 (CC1)
- net at R2.2: now also U12.B5 (CC2)
- net at U1.4 (C-): now also C10.1
- net at U1.6 (C+): now also C10.2
- net ALRT: now reaches U6.5 (ALRT#)
- no-connect marks 4 -> 11
Other:
- added sheet INPUTS (inputs.kicad_sch)
- note added: "PLACE NEXT TO WROOM"
- note added: "SPI FOR PSRAM"
- moved on the sheet: C1, C3, C4, C5, C6, C7, C8, JP1, JP10, JP2, JP3, JP4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

Commit message: and so it begins
Parts:
- added J1: Conn_01x10, Connector_PinHeader_2.54mm:PinHeader_1x10_P2.54mm_Vertical, symbol Connector_Generic:Conn_01x10
Connections:
- net +3.3V: now also J1.2 (Pin_2)
- net +5V: now also J1.3 (Pin_3)
- net ALRT: now also U2.9 (IO16)
- net BTN1: now also U2.6 (IO6)
- net BTN2: now also U2.7 (IO7)
- net ENC_BTN: now also U2.12 (IO8)
- net ENC_SIG_A: now also U2.10 (IO17)
- net ENC_SIG_B: now also U2.11 (IO18)
- net GND: now also J1.1 (Pin_1)
- net PWR_SW: now also U2.8 (IO15)
- net RX: now also J1.5 (Pin_5)
- net TX: now also J1.4 (Pin_4)
- net 21: now reaches U2.23 (IO21)
- net 21: now also J1.8 (Pin_8)
- net 47: now reaches U2.24 (IO47)
- net 47: now also J1.10 (Pin_10)
- net 48: now reaches U2.25 (IO48)
- net 48: now also J1.9 (Pin_9)
- net 02: now reaches U2.38 (IO2)
- net 02: now also J1.7 (Pin_7)
- net 01: now reaches U2.39 (IO1)
- net 01: now also J1.6 (Pin_6)
- no-connect marks 11 -> 17

Commit message: prvni cena test
Parts:
- removed C5: 1uF, new_lib_footprint:C1206, symbol new_lib_symbol:CL31B105KBHNNNE
- added C17: 1uF 0603, new_lib_footprint:C0603, symbol new_lib_symbol:CL10A105KB8NNNC
- JP4: value EXTCOM -> EXTC
- JP8: value EXTMOD -> EXTM
Connections:
- net 47: now also J1.9 (Pin_9); no longer J1.10 (Pin_10)
- net 48: now also J1.10 (Pin_10); no longer J1.9 (Pin_9)
- net GND: now also C17.1
- net RESET: now also C17.2
- no-connect marks 17 -> 18
Changed lines of the file:
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@@
 	)
 	(no_connect
+		(at 78.74 157.48)
+	)
+	(no_connect
 		(at 72.39 181.61)
 	)
@@
 	(wire
 		(pts
-			(xy 104.14 179.07) (xy 106.68 179.07)
-		)
-		(stroke
-			(width 0)
-			(type default)
-		)
-	)
-	(wire
-		(pts
 			(xy 25.4 142.24) (xy 35.56 142.24)
 		)
@@
 	(wire
 		(pts
+			(xy 104.14 181.61) (xy 106.68 181.61)
+		)
+		(stroke
+			(width 0)
+			(type default)
+		)
+	)
+	(wire
+		(pts
 			(xy 195.58 158.75) (xy 196.85 158.75)
 		)
@@
 	(wire
 		(pts
+			(xy 104.14 194.31) (xy 106.68 194.31)
+		)
+		(stroke
+			(width 0)
+			(type default)
+		)
+	)
+	(wire
+		(pts
 			(xy 102.87 171.45) (xy 106.68 171.45)
 		)
@@
 	(wire
 		(pts
+			(xy 104.14 179.07) (xy 106.68 179.07)
+		)
+		(stroke
+			(width 0)
+			(type default)
+		)
+	)
+	(wire
+		(pts
 			(xy 110.49 82.55) (xy 111.76 82.55)
 		)
@@
 	(wire
 		(pts
-			(xy 203.2 109.22) (xy 215.9 109.22)
+			(xy 104.14 191.77) (xy 106.68 191.77)
 		)
 		(stroke
@@
 	(wire
 		(pts
-			(xy 152.4 81.28) (xy 154.94 81.28)
+			(xy 203.2 109.22) (xy 215.9 109.22)
 		)
 		(stroke
@@
 	(wire
 		(pts
-			(xy 236.22 52.07) (xy 238.76 52.07)
+			(xy 152.4 81.28) (xy 154.94 81.28)
 		)
 		(stroke
@@
 	(wire
 		(pts
-			(xy 140.97 45.72) (xy 140.97 48.26)
+			(xy 236.22 52.07) (xy 238.76 52.07)
 		)
 		(stroke
@@
 	(wire
 		(pts
-			(xy 238.76 57.15) (xy 236.22 57.15)
+			(xy 140.97 45.72) (xy 140.97 48.26)
 		)
 		(stroke
@@
 	(wire
 		(pts
-			(xy 68.58 78.74) (xy 69.85 78.74)
+			(xy 238.76 57.15) (xy 236.22 57.15)
 		)
 		(stroke
@@
 	(wire
 		(pts
-			(xy 104.14 181.61) (xy 106.68 181.61)
+			(xy 68.58 78.74) (xy 69.85 78.74)
 		)
 		(stroke
@@
 	(wire
 		(pts
-			(xy 104.14 191.77) (xy 106.68 191.77)
-		)
-		(stroke
-			(width 0)
-			(type default)
-		)
-	)
-	(wire
-		(pts
 			(xy 30.48 50.8) (xy 30.48 53.34)
 		)
@@
 	(wire
 		(pts
-			(xy 104.14 194.31) (xy 106.68 194.31)
-		)
-		(stroke
-			(width 0)
-			(type default)
-		)
-	)
-	(wire
-		(pts
 			(xy 236.22 49.53) (xy 236.22 52.07)
 		)
@@
 	)
 	(label "47"
-		(at 104.14 194.31 0)
+		(at 104.14 191.77 0)
 		(fields_autoplaced yes)
 		(effects
@@
 	)
 	(label "48"
-		(at 104.14 191.77 0)
+		(at 104.14 194.31 0)
 		(fields_autoplaced yes)
 		(effects
@@
 	)
 	(symbol
+		(lib_id "new_lib_symbol:CL10A105KB8NNNC")
+		(at 143.51 179.07 90)
+		(unit 1)
+		(exclude_from_sim no)
+		(in_bom yes)
+		(on_board yes)
+		(dnp no)
+		(fields_autoplaced yes)
+		(property "Reference" "C17"
+			(at 147.32 177.7999 90)
+			(effects
+				(font
+					(size 1.27 1.27)
+				)
+				(justify right)
+			)
+		)
+		(property "Value" "1uF 0603"
+			(at 147.32 180.3399 90)
+			(effects
+				(font
+					(size 1.27 1.27)
+				)
+				(justify right)
+			)
+		)
+		(property "Footprint" "new_lib_footprint:C0603"
+			(at 153.67 179.07 0)
+			(effects
+				(font
+					(size 1.27 1.27)
+					(italic yes)
+				)
+				(hide yes)
+			)
+		)
+		(property "Datasheet" "https://item.szlcsc.com/362304.html"
+			(at 143.383 181.356 0)
+			(effects
+				(font
+					(size 1.27 1.27)
+				)
+				(justify left)
+				(hide yes)
+			)
+		)
+		(property "Description" ""
+			(at 143.51 179.07 0)
+			(effects
+				(font
+					(size 1.27 1.27)
+				)
+				(hide yes)
+			)
+		)
+		(property "LCSC" "C15849"
+			(at 143.51 179.07 0)
+			(effects
+				(font
+					(size 1.27 1.27)
+				)
+				(hide yes)
+			)
+		)
+		(pin "1"
+		)
+		(pin "2"
+		)
+		(instances
+			(project "memory_pcb"
+				(path "/0b554bab-2912-44e0-8d16-f1690413cb05"
+					(reference "C17")
+					(unit 1)
+				)
+			)
+		)
+	)
+	(symbol
 		(lib_id "Jumper:SolderJumper_2_Bridged")
 		(at 242.57 46.99 0)
@@
 			)
 		)
-		(property "Value" "EXTCOM"
-			(at 249.428 46.99 0)
+		(property "Value" "EXTC"
+			(at 244.856 46.99 0)
 			(effects
 				(font
 					(size 1.27 1.27)
 				)
+				(justify left)
 			)
 		)
@@
 		)
 		(property "Value" "VDD"
-			(at 249.428 54.61 0)
+			(at 244.856 54.61 0)
 			(effects
 				(font
 					(size 1.27 1.27)
 				)
+				(justify left)
 			)
 		)
@@
 		)
 		(property "Value" "SCS"
-			(at 249.428 44.45 0)
+			(at 244.856 44.45 0)
 			(effects
 				(font
 					(size 1.27 1.27)
 				)
+				(justify left)
 			)
 		)
@@
 			)
 		)
-		(property "Value" "EXTMOD"
-			(at 249.428 57.15 0)
+		(property "Value" "EXTM"
+			(at 244.856 57.15 0)
 			(effects
 				(font
 					(size 1.27 1.27)
 				)
+				(justify left)
 			)
 		)
@@
 		)
 		(property "Value" "DISP"
-			(at 249.428 49.53 0)
+			(at 244.856 49.53 0)
 			(effects
 				(font
 					(size 1.27 1.27)
 				)
+				(justify left)
 			)
 		)
@@
 	)
 	(symbol
-		(lib_id "new_lib_symbol:CL31B105KBHNNNE")
-		(at 143.51 179.07 90)
-		(unit 1)
-		(exclude_from_sim no)
-		(in_bom yes)
-		(on_board yes)
-		(dnp no)
-		(fields_autoplaced yes)
-		(property "Reference" "C5"
-			(at 147.32 177.7999 90)
-			(effects
-				(font
-					(size 1.27 1.27)
-				)
-				(justify right)
-			)
-		)
-		(property "Value" "1uF"
-			(at 147.32 180.3399 90)
-			(effects
-				(font
-					(size 1.27 1.27)
-				)
-				(justify right)
-			)
-		)
-		(property "Footprint" "new_lib_footprint:C1206"
-			(at 153.67 179.07 0)
-			(effects
-				(font
-					(size 1.27 1.27)
-					(italic yes)
-				)
-				(hide yes)
-			)
-		)
-		(property "Datasheet" "https://item.szlcsc.com/89171.html"
-			(at 143.383 181.356 0)
-			(effects
-				(font
-					(size 1.27 1.27)
-				)
-				(justify left)
-				(hide yes)
-			)
-		)
-		(property "Description" ""
-			(at 143.51 179.07 0)
-			(effects
-				(font
-					(size 1.27 1.27)
-				)
-				(hide yes)
-			)
-		)
-		(property "LCSC" "C1848"
-			(at 143.51 179.07 0)
-			(effects
-				(font
-					(size 1.27 1.27)
-				)
-				(hide yes)
-			)
-		)
-		(pin "2"
-		)
-		(pin "1"
-		)
-		(instances
-			(project "memory_pcb"
-				(path "/0b554bab-2912-44e0-8d16-f1690413cb05"
-					(reference "C5")
-					(unit 1)
-				)
-			)
-		)
-	)
-	(symbol
 		(lib_id "new_lib_symbol:0402B102K500NT")
 		(at 144.78 121.92 270)
@@
 		)
 		(property "Value" "VSS"
-			(at 249.428 59.69 0)
+			(at 244.856 59.69 0)
 			(effects
 				(font
 					(size 1.27 1.27)
 				)
+				(justify left)
 			)
 		)
@@
 		)
 		(property "Value" "VSSA"
-			(at 249.428 62.23 0)
+			(at 244.856 62.23 0)
 			(effects
 				(font
 					(size 1.27 1.27)
 				)
+				(justify left)
 			)
 		)
@@
 		)
 		(property "Value" "MOSI"
-			(at 249.428 41.91 0)
+			(at 244.856 41.91 0)
 			(effects
 				(font
 					(size 1.27 1.27)
 				)
+				(justify left)
 			)
 		)
@@
 		)
 		(property "Value" "VDDA"
-			(at 249.428 52.07 0)
+			(at 244.856 52.07 0)
 			(effects
 				(font
 					(size 1.27 1.27)
 				)
+				(justify left)
 			)
 		)
@@
 		)
 		(property "Value" "CKL"
-			(at 249.428 39.37 0)
+			(at 244.856 39.37 0)
 			(effects
 				(font
 					(size 1.27 1.27)
 				)
+				(justify left)
 			)
 		)

Commit message: uz nevim, dneska asi konec
Parts:
- U5: value BOOT -> TS-1088-AR02016
Changed lines of the file:
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@@
 			)
 		)
-		(property "Value" "BOOT"
+		(property "Value" "TS-1088-AR02016"
 			(at 160.782 167.132 0)
 			(effects

Commit message: im sleeping
Connections:
- net 21: now also J1.10 (Pin_10); no longer J1.8 (Pin_8)
- net 48: now also J1.8 (Pin_8); no longer J1.10 (Pin_10)

Commit message: looks rdy
Parts:
- removed C12: 1uF, new_lib_footprint:C1206, symbol new_lib_symbol:CL31B105KBHNNNE
- added C5: 1uF 0603, new_lib_footprint:C0603, symbol new_lib_symbol:CL10A105KB8NNNC
- added TP1: D+, TestPoint:TestPoint_Pad_D1.0mm, symbol Connector:TestPoint
- added TP2: D-, TestPoint:TestPoint_Pad_D1.0mm, symbol Connector:TestPoint
- R3, R8, R9: value 5.1kOhm -> 10kOhm; LCSC C23186 -> C25804
- renumbered U5 to SW1, U4 to SW2
Connections:
- net +3.3V: now also C5.1
- net D+: now also TP1.1
- net D-: now also TP2.1
- net GND: now also SW1.2, C5.2; no longer SW1.1
- net BOOT: no longer names the net of U2.27 (IO0)
- net BOOT: now also SW1.1; no longer SW1.2
- net RESET: no longer names the net of C17.2, R3.1, SW2.2, U2.3 (EN)
Other:
- moved on the sheet: C1, C13, C17, C9, H1, H2, H3, H4, J1, R3, R8, R9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

Commit message: :)
Parts:
- added C12, C18: 0.1uF, new_lib_footprint:C0402, symbol new_lib_symbol:CL05B104KO5NNNC
- added C19: 1uF 0603, new_lib_footprint:C0603, symbol new_lib_symbol:CL10A105KB8NNNC
Connections:
- net +5V: now also C18.2, C19.1; no longer JP5.1 (A), JP7.1 (A)
- net GND: now also C12.1, C18.1, C19.2; no longer JP8.1 (A)
- net DISP_ON: now reaches U2.31 (IO38)
- net DISP_ON: now also JP5.1 (A), C12.2
- no-connect marks 18 -> 17
Other:
- moved on the sheet: JP1, JP10, JP2, JP3, JP4, JP5, JP6, JP7, JP8, JP9, P1

Commit message: a
Connections:
- net +5V: now also JP7.1 (A)
- net GND: now also JP8.1 (A)
Other:
- moved on the sheet: TP2
Changed lines of the file:
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@@
 	)
 	(junction
+		(at 248.92 146.05)
+		(diameter 0)
+		(color 0 0 0 0)
+	)
+	(junction
 		(at 199.39 149.86)
 		(diameter 0)
@@
 	)
 	(junction
+		(at 245.11 46.99)
+		(diameter 0)
+		(color 0 0 0 0)
+	)
+	(junction
 		(at 66.04 40.64)
 		(diameter 0)
@@
 	)
 	(junction
-		(at 247.65 146.05)
+		(at 245.11 39.37)
 		(diameter 0)
 		(color 0 0 0 0)
@@
 	(wire
 		(pts
-			(xy 247.65 140.97) (xy 260.35 140.97)
+			(xy 248.92 140.97) (xy 260.35 140.97)
 		)
 		(stroke
@@
 	(wire
 		(pts
+			(xy 245.11 39.37) (xy 245.11 41.91)
+		)
+		(stroke
+			(width 0)
+			(type default)
+		)
+	)
+	(wire
+		(pts
 			(xy 156.21 43.18) (xy 157.48 43.18)
 		)
@@
 	(wire
 		(pts
+			(xy 247.65 138.43) (xy 254 138.43)
+		)
+		(stroke
+			(width 0)
+			(type default)
+		)
+	)
+	(wire
+		(pts
 			(xy 41.91 162.56) (xy 52.07 162.56)
 		)
@@
 	(wire
 		(pts
+			(xy 245.11 44.45) (xy 245.11 46.99)
+		)
+		(stroke
+			(width 0)
+			(type default)
+		)
+	)
+	(wire
+		(pts
 			(xy 27.94 110.49) (xy 38.1 110.49)
 		)
@@
 	(wire
 		(pts
-			(xy 247.65 146.05) (xy 260.35 146.05)
+			(xy 247.65 146.05) (xy 248.92 146.05)
 		)
 		(stroke
@@
 	(wire
 		(pts
-			(xy 247.65 140.97) (xy 247.65 146.05)
+			(xy 248.92 140.97) (xy 248.92 146.05)
 		)
 		(stroke
@@
 		)
 	)
+	(wire
+		(pts
+			(xy 248.92 146.05) (xy 260.35 146.05)
+		)
+		(stroke
+			(width 0)
+			(type default)
+		)
+	)
 	(text "SPI FOR PSRAM\n"
 		(exclude_from_sim no)
@@
 	(symbol
 		(lib_id "Connector:TestPoint")
-		(at 254 138.43 90)
+		(at 247.65 138.43 90)
 		(unit 1)
 		(exclude_from_sim no)
@@
 		(dnp no)
 		(property "Reference" "TP2"
-			(at 244.094 138.43 90)
+			(at 237.744 138.43 90)
 			(effects
 				(font
@@
 		)
 		(property "Value" "D-"
-			(at 247.65 138.43 90)
+			(at 241.3 138.43 90)
 			(effects
 				(font
@@
 		)
 		(property "Footprint" "TestPoint:TestPoint_Pad_D1.0mm"
-			(at 254 133.35 0)
+			(at 247.65 133.35 0)
 			(effects
 				(font
@@
 		)
 		(property "Datasheet" "~"
-			(at 254 133.35 0)
+			(at 247.65 133.35 0)
 			(effects
 				(font
@@
 		)
 		(property "Description" "test point"
-			(at 254 138.43 0)
+			(at 247.65 138.43 0)
 			(effects
 				(font
