File: memory_pcb/memory_pcb.kicad_sch (KiCad schematic)
At the start: 53 parts, among them J1 Conn_01x10, P1 AFC01-S10FCC-00, SW1 TS-1088-AR02016, SW2 TS-1088-AR02016, U1 AP3602AKTR-G1 SETUPUP, U10 DMG3415U, U11 SS54_C22452, U12 TYPE-C-31-M-12, U2 ESP32-S3-WROOM-1(N16R8), U6 MAX17048G+T10 FUEL GAUGE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

Commit message: posilam
Parts:
- removed TP1: D+, TestPoint:TestPoint_Pad_D1.0mm, symbol Connector:TestPoint
- removed TP2: D-, TestPoint:TestPoint_Pad_D1.0mm, symbol Connector:TestPoint
Connections:
- net +3.3V: now also J1.3 (Pin_3); no longer J1.2 (Pin_2)
- net +5V: now also J1.2 (Pin_2); no longer J1.3 (Pin_3)
Changed lines of the file:
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@@
 	)
 	(junction
-		(at 248.92 146.05)
-		(diameter 0)
-		(color 0 0 0 0)
-	)
-	(junction
 		(at 199.39 149.86)
 		(diameter 0)
@@
 	)
 	(junction
-		(at 254 138.43)
-		(diameter 0)
-		(color 0 0 0 0)
-	)
-	(junction
 		(at 245.11 39.37)
 		(diameter 0)
@@
 	(wire
 		(pts
-			(xy 247.65 138.43) (xy 254 138.43)
-		)
-		(stroke
-			(width 0)
-			(type default)
-		)
-	)
-	(wire
-		(pts
 			(xy 41.91 162.56) (xy 52.07 162.56)
 		)
@@
 	(wire
 		(pts
-			(xy 114.3 102.87) (xy 118.11 102.87)
-		)
-		(stroke
-			(width 0)
-			(type default)
-		)
-	)
-	(wire
-		(pts
 			(xy 176.53 129.54) (xy 176.53 132.08)
 		)
@@
 	(wire
 		(pts
-			(xy 247.65 146.05) (xy 248.92 146.05)
-		)
-		(stroke
-			(width 0)
-			(type default)
-		)
-	)
-	(wire
-		(pts
 			(xy 40.64 83.82) (xy 36.83 83.82)
 		)
@@
 	(wire
 		(pts
+			(xy 114.3 102.87) (xy 118.11 102.87)
+		)
+		(stroke
+			(width 0)
+			(type default)
+		)
+	)
+	(wire
+		(pts
 			(xy 40.64 83.82) (xy 45.72 83.82)
 		)
@@
 	(wire
 		(pts
-			(xy 257.81 130.81) (xy 260.35 130.81)
+			(xy 114.3 105.41) (xy 118.11 105.41)
 		)
 		(stroke
@@
 	(wire
 		(pts
-			(xy 22.86 107.95) (xy 22.86 110.49)
+			(xy 257.81 130.81) (xy 260.35 130.81)
 		)
 		(stroke
@@
 	(wire
 		(pts
-			(xy 74.93 43.18) (xy 74.93 40.64)
+			(xy 22.86 107.95) (xy 22.86 110.49)
 		)
 		(stroke
@@
 	(wire
 		(pts
-			(xy 114.3 105.41) (xy 118.11 105.41)
+			(xy 74.93 43.18) (xy 74.93 40.64)
 		)
 		(stroke
@@
 	)
 	(symbol
-		(lib_id "Connector:TestPoint")
-		(at 247.65 146.05 90)
-		(unit 1)
-		(exclude_from_sim no)
-		(in_bom yes)
-		(on_board yes)
-		(dnp no)
-		(property "Reference" "TP1"
-			(at 237.744 146.05 90)
-			(effects
-				(font
-					(size 1.27 1.27)
-				)
-			)
-		)
-		(property "Value" "D+"
-			(at 241.3 146.05 90)
-			(effects
-				(font
-					(size 1.27 1.27)
-				)
-			)
-		)
-		(property "Footprint" "TestPoint:TestPoint_Pad_D1.0mm"
-			(at 247.65 140.97 0)
-			(effects
-				(font
-					(size 1.27 1.27)
-				)
-				(hide yes)
-			)
-		)
-		(property "Datasheet" "~"
-			(at 247.65 140.97 0)
-			(effects
-				(font
-					(size 1.27 1.27)
-				)
-				(hide yes)
-			)
-		)
-		(property "Description" "test point"
-			(at 247.65 146.05 0)
-			(effects
-				(font
-					(size 1.27 1.27)
-				)
-				(hide yes)
-			)
-		)
-		(pin "1"
-		)
-		(instances
-			(project "memory_pcb"
-				(path "/0b554bab-2912-44e0-8d16-f1690413cb05"
-					(reference "TP1")
-					(unit 1)
-				)
-			)
-		)
-	)
-	(symbol
 		(lib_id "new_lib_symbol:0603WAF5101T5E")
 		(at 243.84 135.89 0)
@@
 	(symbol
 		(lib_id "power:+5V")
-		(at 114.3 105.41 90)
+		(at 114.3 102.87 90)
 		(unit 1)
 		(exclude_from_sim no)
@@
 		(fields_autoplaced yes)
 		(property "Reference" "#PWR071"
-			(at 118.11 105.41 0)
+			(at 118.11 102.87 0)
 			(effects
 				(font
@@
 		)
 		(property "Value" "+5V"
-			(at 110.49 105.4099 90)
+			(at 110.49 102.8699 90)
 			(effects
 				(font
@@
 		)
 		(property "Footprint" ""
-			(at 114.3 105.41 0)
+			(at 114.3 102.87 0)
 			(effects
 				(font
@@
 		)
 		(property "Datasheet" ""
-			(at 114.3 105.41 0)
+			(at 114.3 102.87 0)
 			(effects
 				(font
@@
 		)
 		(property "Description" "Power symbol creates a global label with name \"+5V\""
-			(at 114.3 105.41 0)
+			(at 114.3 102.87 0)
 			(effects
 				(font
@@
 	)
 	(symbol
-		(lib_id "Connector:TestPoint")
-		(at 247.65 138.43 90)
-		(unit 1)
-		(exclude_from_sim no)
-		(in_bom yes)
-		(on_board yes)
-		(dnp no)
-		(property "Reference" "TP2"
-			(at 237.744 138.43 90)
-			(effects
-				(font
-					(size 1.27 1.27)
-				)
-			)
-		)
-		(property "Value" "D-"
-			(at 241.3 138.43 90)
-			(effects
-				(font
-					(size 1.27 1.27)
-				)
-			)
-		)
-		(property "Footprint" "TestPoint:TestPoint_Pad_D1.0mm"
-			(at 247.65 133.35 0)
-			(effects
-				(font
-					(size 1.27 1.27)
-				)
-				(hide yes)
-			)
-		)
-		(property "Datasheet" "~"
-			(at 247.65 133.35 0)
-			(effects
-				(font
-					(size 1.27 1.27)
-				)
-				(hide yes)
-			)
-		)
-		(property "Description" "test point"
-			(at 247.65 138.43 0)
-			(effects
-				(font
-					(size 1.27 1.27)
-				)
-				(hide yes)
-			)
-		)
-		(pin "1"
-		)
-		(instances
-			(project "memory_pcb"
-				(path "/0b554bab-2912-44e0-8d16-f1690413cb05"
-					(reference "TP2")
-					(unit 1)
-				)
-			)
-		)
-	)
-	(symbol
 		(lib_id "new_lib_symbol:0603WAF5101T5E")
 		(at 22.86 102.87 90)
@@
 	(symbol
 		(lib_id "power:+3.3V")
-		(at 114.3 102.87 90)
+		(at 114.3 105.41 90)
 		(unit 1)
 		(exclude_from_sim no)
@@
 		(on_board yes)
 		(dnp no)
-		(fields_autoplaced yes)
 		(property "Reference" "#PWR069"
-			(at 118.11 102.87 0)
+			(at 118.11 105.41 0)
 			(effects
 				(font
@@
 		)
 		(property "Value" "+3.3V"
-			(at 110.49 102.8699 90)
+			(at 110.49 105.4099 90)
 			(effects
 				(font
@@
 		)
 		(property "Footprint" ""
-			(at 114.3 102.87 0)
+			(at 114.3 105.41 0)
 			(effects
 				(font
@@
 		)
 		(property "Datasheet" ""
-			(at 114.3 102.87 0)
+			(at 114.3 105.41 0)
 			(effects
 				(font
@@
 		)
 		(property "Description" "Power symbol creates a global label with name \"+3.3V\""
-			(at 114.3 102.87 0)
+			(at 114.3 105.41 0)
 			(effects
 				(font
